Commit message: chore: working CLI

File: src/defined_description/urdf/defined_mvp.urdf.xacro (robot description, xacro)
@@ -28,5 +28,5 @@
   <xacro:property name="wheel_mass"       value="0.1"/>
   <xacro:property name="wheel_separation" value="0.287"/>
-  <xacro:property name="caster_radius"    value="0.010"/>
+  <xacro:property name="caster_radius"    value="0.020"/>
   <xacro:property name="caster_mass"      value="0.05"/>
   <!-- Derived offsets -->
@@ -130,5 +130,5 @@
       <parent link="base_link"/>
       <child  link="${side}_wheel_link"/>
-      <origin xyz="0 ${y_sign * wheel_y} ${wheel_z}" rpy="0 0 0"/>
+      <origin xyz="-0.08 ${y_sign * wheel_y} ${wheel_z}" rpy="0 0 0"/>
       <axis xyz="0 1 0"/>
     </joint>
@@ -168,7 +168,9 @@
   </joint>
   <gazebo reference="caster_link">
-    <!-- Zero friction so caster slides freely -->
+    <!-- Zero friction so caster slides freely; stiff contact to prevent bouncing -->
     <mu1>0.0</mu1>
     <mu2>0.0</mu2>
+    <kp>1000000.0</kp>
+    <kd>100.0</kd>
   </gazebo>
   <!-- ============================================================
@@ -219,5 +221,5 @@
         </scan>
         <range>
-          <min>0.12</min>
+          <min>0.20</min>
           <max>3.5</max>
           <resolution>0.01</resolution>
