Commit message: feat: migrate to Gz Sim (Ionic) + ROS Jazzy with Nav2 and SLAM
- Migrate from Gazebo Classic to Gz Sim: SDF 1.9 worlds, gz-sim plugins
- Update URDF for Gz Sim (gpu_lidar, gz-sim-*-system plugins, gz_frame_id)
- Docker: ROS Jazzy base, non-root user, security hardening, healthcheck
- Nav2 config updated for Jazzy plugin names (:: separator)
- SLAM toolbox with separate lifecycle manager (bond_timeout: 0.0)
- Gz bridge config (YAML) for ros_gz_bridge topic bridging
- BT tree XML collection for Nav2 navigation behaviors
- Move simulation docs to docs/simulation.md

Co-Authored-By: Claude Opus 4.6 <noreply@anthropic.com>

File: src/defined_description/urdf/defined_mvp.urdf.xacro (robot description, xacro)
@@ -10,7 +10,9 @@
     Wheels : cylinder radius=0.033 m, width=0.020 m  (left + right)
     Caster : sphere  radius=0.010 m  (front, passive)
-  Gazebo plugins:
-    libgazebo_ros_diff_drive           → /cmd_vel, /odom, odom→base_footprint TF
-    libgazebo_ros_joint_state_publisher → /joint_states
+  Gz Sim plugins (declared in URDF <gazebo> blocks, converted to SDF by ros_gz):
+    gz-sim-diff-drive-system        → subscribes /cmd_vel, publishes /odom (Gz topics)
+    gz-sim-joint-state-publisher-system → publishes /joint_states (Gz topic)
+    Lidar sensor                    → publishes /scan (Gz topic)
+  All Gz topics are bridged to ROS2 by ros_gz_bridge in gazebo.launch.py.
 -->
 <robot xmlns:xacro="http://www.ros.org/wiki/xacro" name="defined_mvp">
@@ -97,7 +99,4 @@
                        x="${base_length}" y="${base_width}" z="${base_height}"/>
   </link>
-  <gazebo reference="base_link">
-    <material>Gazebo/Blue</material>
-  </gazebo>
   <!-- ============================================================
        WHEEL MACRO
@@ -132,5 +131,5 @@
       <axis xyz="0 1 0"/>
     </joint>
-    <!-- Gazebo: high friction so wheels grip the floor -->
+    <!-- Gz: high friction so wheels grip the floor -->
     <gazebo reference="${side}_wheel_link">
       <mu1>1.0</mu1>
@@ -138,5 +137,4 @@
       <kp>1000000.0</kp>
       <kd>100.0</kd>
-      <material>Gazebo/DarkGrey</material>
     </gazebo>
   </xacro:macro>
@@ -171,10 +169,9 @@
     <mu1>0.0</mu1>
     <mu2>0.0</mu2>
-    <material>Gazebo/Grey</material>
   </gazebo>
   <!-- ============================================================
        LIDAR — 2D laser scanner on top of base
        360° scan, 0.12–3.5 m range, ~5.5 Hz, 360 samples
-       Publishes sensor_msgs/LaserScan on /scan
+       Publishes to Gz topic /scan (bridged to ROS2 by ros_gz_bridge)
        ============================================================ -->
   <xacro:property name="lidar_radius" value="0.030"/>
@@ -204,9 +201,10 @@
   </joint>
   <gazebo reference="lidar_link">
-    <material>Gazebo/Black</material>
-    <sensor type="ray" name="lidar_sensor">
+    <sensor type="gpu_lidar" name="lidar_sensor">
       <pose>0 0 0 0 0 0</pose>
       <visualize>true</visualize>
       <update_rate>5.5</update_rate>
+      <topic>/scan</topic>
+      <gz_frame_id>lidar_link</gz_frame_id>
       <ray>
         <scan>
@@ -229,50 +227,40 @@
         </noise>
       </ray>
-      <plugin name="gazebo_ros_lidar" filename="libgazebo_ros_ray_sensor.so">
-        <ros>
-          <remapping>~/out:=scan</remapping>
-        </ros>
-        <output_type>sensor_msgs/LaserScan</output_type>
-        <frame_name>lidar_link</frame_name>
-      </plugin>
     </sensor>
   </gazebo>
   <!-- ============================================================
-       GAZEBO PLUGIN: DIFFERENTIAL DRIVE
-       Subscribes : /cmd_vel  (geometry_msgs/Twist)
-       Publishes  : /odom     (nav_msgs/Odometry)
-       Broadcasts : odom → base_footprint TF
+       GZ SIM PLUGIN: DIFFERENTIAL DRIVE
+       Subscribes : /cmd_vel  (gz.msgs.Twist)
+       Publishes  : /odom     (gz.msgs.Odometry)
+       Broadcasts : odom → base_footprint TF (via ros_gz_bridge)
        ============================================================ -->
   <gazebo>
-    <plugin name="diff_drive_controller" filename="libgazebo_ros_diff_drive.so">
-      <update_rate>50</update_rate>
+    <plugin filename="gz-sim-diff-drive-system" name="gz::sim::systems::DiffDrive">
       <left_joint>left_wheel_joint</left_joint>
       <right_joint>right_wheel_joint</right_joint>
       <!-- Must match RDF yaml values -->
       <wheel_separation>${wheel_separation}</wheel_separation>
-      <wheel_diameter>${2.0 * wheel_radius}</wheel_diameter>
-      <max_wheel_torque>20</max_wheel_torque>
-      <max_wheel_acceleration>1.0</max_wheel_acceleration>
-      <command_topic>cmd_vel</command_topic>
-      <odometry_topic>odom</odometry_topic>
-      <odometry_frame>odom</odometry_frame>
-      <robot_base_frame>base_footprint</robot_base_frame>
-      <publish_odom>true</publish_odom>
-      <publish_odom_tf>true</publish_odom_tf>
-      <!-- TF for wheel joints comes from joint_state_publisher + robot_state_publisher -->
-      <publish_wheel_tf>false</publish_wheel_tf>
+      <wheel_radius>${wheel_radius}</wheel_radius>
+      <max_linear_acceleration>1.0</max_linear_acceleration>
+      <topic>/cmd_vel</topic>
+      <odom_topic>/odom</odom_topic>
+      <frame_id>odom</frame_id>
+      <child_frame_id>base_footprint</child_frame_id>
+      <odom_publish_frequency>50</odom_publish_frequency>
+      <tf_topic>/tf</tf_topic>
     </plugin>
   </gazebo>
   <!-- ============================================================
-       GAZEBO PLUGIN: JOINT STATE PUBLISHER
-       Publishes  : /joint_states (sensor_msgs/JointState)
-       Required by robot_state_publisher to compute wheel TF.
+       GZ SIM PLUGIN: JOINT STATE PUBLISHER
+       Publishes  : /world/<world>/model/defined_mvp/joint_state (gz topic)
+       Bridged to /joint_states by ros_gz_bridge.
        ============================================================ -->
   <gazebo>
-    <plugin name="gazebo_joint_state_publisher"
-            filename="libgazebo_ros_joint_state_publisher.so">
-      <update_rate>50</update_rate>
+    <plugin filename="gz-sim-joint-state-publisher-system"
+            name="gz::sim::systems::JointStatePublisher">
       <joint_name>left_wheel_joint</joint_name>
       <joint_name>right_wheel_joint</joint_name>
+      <update_rate>50</update_rate>
+      <topic>/joint_states</topic>
     </plugin>
   </gazebo>

Commit message: fix(description): update URDF for Gz Sim compatibility
Co-Authored-By: Claude Opus 4.6 <noreply@anthropic.com>

File: src/defined_description/urdf/defined_mvp.urdf.xacro (robot description, xacro)
@@ -35,7 +35,7 @@
   <!-- Wheel Z relative to base_link centre; wheel tangent at base bottom -->
   <xacro:property name="wheel_z"   value="${-base_height / 2.0}"/>
-  <!-- Caster at front edge of base, level with ground -->
+  <!-- Caster at front edge of base, bottom touching ground -->
   <xacro:property name="caster_x"  value="${base_length / 2.0 - caster_radius}"/>
-  <xacro:property name="caster_z"  value="${-base_height / 2.0 - caster_radius}"/>
+  <xacro:property name="caster_z"  value="${-(base_height / 2.0 + wheel_radius - caster_radius)}"/>
   <!-- ============================================================
        INERTIA HELPERS
@@ -76,6 +76,8 @@
     <parent link="base_footprint"/>
     <child  link="base_link"/>
-    <!-- Lift base_link centre to wheel_radius above ground -->
-    <origin xyz="0 0 ${wheel_radius}" rpy="0 0 0"/>
+    <!-- Lift base_link centre so wheel axles are at ground level:
+         base_link_z = base_height/2 + wheel_radius
+         This ensures wheel bottoms touch ground and caster contacts ground. -->
+    <origin xyz="0 0 ${base_height / 2.0 + wheel_radius}" rpy="0 0 0"/>
   </joint>
   <!-- ============================================================
@@ -172,5 +174,5 @@
   <!-- ============================================================
        LIDAR — 2D laser scanner on top of base
-       360° scan, 0.12–3.5 m range, ~5.5 Hz, 360 samples
+       360° scan, 0.12–3.5 m range, ~20 Hz, 720 samples
        Publishes to Gz topic /scan (bridged to ROS2 by ros_gz_bridge)
        ============================================================ -->
@@ -204,5 +206,5 @@
       <pose>0 0 0 0 0 0</pose>
       <visualize>true</visualize>
-      <update_rate>5.5</update_rate>
+      <update_rate>20</update_rate>
       <topic>/scan</topic>
       <gz_frame_id>lidar_link</gz_frame_id>
@@ -210,5 +212,5 @@
         <scan>
           <horizontal>
-            <samples>360</samples>
+            <samples>720</samples>
             <resolution>1</resolution>
             <min_angle>-3.14159265359</min_angle>
@@ -224,5 +226,5 @@
           <type>gaussian</type>
           <mean>0.0</mean>
-          <stddev>0.01</stddev>
+          <stddev>0.0</stddev>
         </noise>
       </ray>
@@ -233,5 +235,5 @@
        Subscribes : /cmd_vel  (gz.msgs.Twist)
        Publishes  : /odom     (gz.msgs.Odometry)
-       Broadcasts : odom → base_footprint TF (via ros_gz_bridge)
+       TF odom→base_footprint: published by odom_tf_broadcaster.py from /odom
        ============================================================ -->
   <gazebo>
@@ -248,5 +250,5 @@
       <child_frame_id>base_footprint</child_frame_id>
       <odom_publish_frequency>50</odom_publish_frequency>
-      <tf_topic>/tf</tf_topic>
+      <tf_topic>/odom_tf</tf_topic>
     </plugin>
   </gazebo>

Commit message: feat(platform): parametric xacro and Nav2 overrides from ROBOT_* env vars (DR-022)
URDF is now conditional on has_lidar/has_camera args. Lidar specs,
camera config, and Nav2 velocity limits are driven by env vars set
from RDF via the CLI. Backward-compatible defaults match existing model.

Co-Authored-By: Claude Opus 4.6 <noreply@anthropic.com>

File: src/defined_description/urdf/defined_mvp.urdf.xacro (robot description, xacro)
@@ -18,4 +18,22 @@
 <robot xmlns:xacro="http://www.ros.org/wiki/xacro" name="defined_mvp">
   <!-- ============================================================
+       XACRO ARGS — overridable from launch (populated from ROBOT_* env vars)
+       All have backward-compatible defaults matching the original URDF.
+       NOTE: wheel_separation/wheel_radius are accepted for interface
+       compatibility but NOT used — physical geometry and diff-drive
+       odometry both use the hardcoded properties below.
+       ============================================================ -->
+  <xacro:arg name="wheel_separation"  default="0.287"/>
+  <xacro:arg name="wheel_radius"      default="0.033"/>
+  <xacro:arg name="has_lidar"         default="true"/>
+  <xacro:arg name="lidar_range_min"   default="0.20"/>
+  <xacro:arg name="lidar_range_max"   default="3.5"/>
+  <xacro:arg name="lidar_samples"     default="720"/>
+  <xacro:arg name="lidar_update_rate" default="20"/>
+  <xacro:arg name="has_camera"        default="false"/>
+  <xacro:arg name="camera_width"      default="640"/>
+  <xacro:arg name="camera_height"     default="480"/>
+  <xacro:arg name="camera_fps"        default="30"/>
+  <!-- ============================================================
        PROPERTIES
        ============================================================ -->
@@ -24,4 +42,7 @@
   <xacro:property name="base_height"      value="0.10"/>
   <xacro:property name="base_mass"        value="2.0"/>
+  <!-- Physical geometry values — fixed to match this URDF's visual model.
+       The RDF wheel_separation/radius args are used ONLY by the diff-drive
+       plugin for odometry, not for joint positions or visual geometry. -->
   <xacro:property name="wheel_radius"     value="0.033"/>
   <xacro:property name="wheel_width"      value="0.020"/>
@@ -175,62 +196,127 @@
   </gazebo>
   <!-- ============================================================
-       LIDAR — 2D laser scanner on top of base
-       360° scan, 0.12–3.5 m range, ~20 Hz, 720 samples
+       LIDAR — conditional 2D laser scanner on top of base
+       Controlled by has_lidar arg (default: true).
+       Parameters driven by lidar_* args from ROBOT_* env vars.
        Publishes to Gz topic /scan (bridged to ROS2 by ros_gz_bridge)
        ============================================================ -->
-  <xacro:property name="lidar_radius" value="0.030"/>
-  <xacro:property name="lidar_height" value="0.020"/>
-  <xacro:property name="lidar_mass"   value="0.1"/>
-  <link name="lidar_link">
-    <visual>
-      <geometry>
-        <cylinder radius="${lidar_radius}" length="${lidar_height}"/>
-      </geometry>
-      <material name="lidar_black">
-        <color rgba="0.1 0.1 0.1 1.0"/>
-      </material>
-    </visual>
-    <collision>
-      <geometry>
-        <cylinder radius="${lidar_radius}" length="${lidar_height}"/>
-      </geometry>
-    </collision>
-    <xacro:cylinder_inertia m="${lidar_mass}" r="${lidar_radius}" h="${lidar_height}"/>
-  </link>
-  <joint name="lidar_joint" type="fixed">
-    <parent link="base_link"/>
-    <child  link="lidar_link"/>
-    <!-- Centred on top of the base box -->
-    <origin xyz="0 0 ${base_height / 2.0 + lidar_height / 2.0}" rpy="0 0 0"/>
-  </joint>
-  <gazebo reference="lidar_link">
-    <sensor type="gpu_lidar" name="lidar_sensor">
-      <pose>0 0 0 0 0 0</pose>
-      <visualize>true</visualize>
-      <update_rate>20</update_rate>
-      <topic>/scan</topic>
-      <gz_frame_id>lidar_link</gz_frame_id>
-      <ray>
-        <scan>
-          <horizontal>
-            <samples>720</samples>
-            <resolution>1</resolution>
-            <min_angle>-3.14159265359</min_angle>
-            <max_angle>3.14159265359</max_angle>
-          </horizontal>
-        </scan>
-        <range>
-          <min>0.20</min>
-          <max>3.5</max>
-          <resolution>0.01</resolution>
-        </range>
-        <noise>
-          <type>gaussian</type>
-          <mean>0.0</mean>
-          <stddev>0.0</stddev>
-        </noise>
-      </ray>
-    </sensor>
-  </gazebo>
+  <xacro:if value="$(arg has_lidar)">
+    <xacro:property name="lidar_radius" value="0.030"/>
+    <xacro:property name="lidar_height" value="0.020"/>
+    <xacro:property name="lidar_mass"   value="0.1"/>
+    <link name="lidar_link">
+      <visual>
+        <geometry>
+          <cylinder radius="${lidar_radius}" length="${lidar_height}"/>
+        </geometry>
+        <material name="lidar_black">
+          <color rgba="0.1 0.1 0.1 1.0"/>
+        </material>
+      </visual>
+      <collision>
+        <geometry>
+          <cylinder radius="${lidar_radius}" length="${lidar_height}"/>
+        </geometry>
+      </collision>
+      <xacro:cylinder_inertia m="${lidar_mass}" r="${lidar_radius}" h="${lidar_height}"/>
+    </link>
+    <joint name="lidar_joint" type="fixed">
+      <parent link="base_link"/>
+      <child  link="lidar_link"/>
+      <!-- Centred on top of the base box -->
+      <origin xyz="0 0 ${base_height / 2.0 + lidar_height / 2.0}" rpy="0 0 0"/>
+    </joint>
+    <gazebo reference="lidar_link">
+      <sensor type="gpu_lidar" name="lidar_sensor">
+        <pose>0 0 0 0 0 0</pose>
+        <visualize>true</visualize>
+        <update_rate>$(arg lidar_update_rate)</update_rate>
+        <topic>/scan</topic>
+        <gz_frame_id>lidar_link</gz_frame_id>
+        <ray>
+          <scan>
+            <horizontal>
+              <samples>$(arg lidar_samples)</samples>
+              <resolution>1</resolution>
+              <min_angle>-3.14159265359</min_angle>
+              <max_angle>3.14159265359</max_angle>
+            </horizontal>
+          </scan>
+          <range>
+            <min>$(arg lidar_range_min)</min>
+            <max>$(arg lidar_range_max)</max>
+            <resolution>0.01</resolution>
+          </range>
+          <noise>
+            <type>gaussian</type>
+            <mean>0.0</mean>
+            <stddev>0.0</stddev>
+          </noise>
+        </ray>
+      </sensor>
+    </gazebo>
+  </xacro:if>
+  <!-- ============================================================
+       CAMERA — conditional RGB camera on front of base
+       Controlled by has_camera arg (default: false).
+       Parameters driven by camera_* args from ROBOT_* env vars.
+       Publishes to Gz topic /camera/image_raw (bridged to ROS2)
+       ============================================================ -->
+  <xacro:if value="$(arg has_camera)">
+    <xacro:property name="camera_box_size" value="0.02"/>
+    <xacro:property name="camera_mass"     value="0.05"/>
+    <link name="camera_link">
+      <visual>
+        <geometry>
+          <box size="${camera_box_size} ${camera_box_size * 2} ${camera_box_size}"/>
+        </geometry>
+        <material name="camera_grey">
+          <color rgba="0.3 0.3 0.3 1.0"/>
+        </material>
+      </visual>
+      <collision>
+        <geometry>
+          <box size="${camera_box_size} ${camera_box_size * 2} ${camera_box_size}"/>
+        </geometry>
+      </collision>
+      <xacro:box_inertia m="${camera_mass}"
+                         x="${camera_box_size}" y="${camera_box_size * 2}" z="${camera_box_size}"/>
+    </link>
+    <!-- Camera optical frame: Z forward, X right, Y down (ROS convention) -->
+    <link name="camera_optical_link"/>
+    <joint name="camera_joint" type="fixed">
+      <parent link="base_link"/>
+      <child  link="camera_link"/>
+      <!-- Front-centre of base, slightly above centre -->
+      <origin xyz="${base_length / 2.0} 0 ${base_height / 4.0}" rpy="0 0 0"/>
+    </joint>
+    <joint name="camera_optical_joint" type="fixed">
+      <parent link="camera_link"/>
+      <child  link="camera_optical_link"/>
+      <!-- Rotate from URDF (X-forward) to optical (Z-forward) convention -->
+      <origin xyz="0 0 0" rpy="${-pi/2} 0 ${-pi/2}"/>
+    </joint>
+    <gazebo reference="camera_link">
+      <sensor type="camera" name="camera_sensor">
+        <pose>0 0 0 0 0 0</pose>
+        <visualize>true</visualize>
+        <update_rate>$(arg camera_fps)</update_rate>
+        <topic>/camera/image_raw</topic>
+        <gz_frame_id>camera_optical_link</gz_frame_id>
+        <camera>
+          <horizontal_fov>1.3962634</horizontal_fov>
+          <image>
+            <width>$(arg camera_width)</width>
+            <height>$(arg camera_height)</height>
+            <format>R8G8B8</format>
+          </image>
+          <clip>
+            <near>0.02</near>
+            <far>100</far>
+          </clip>
+        </camera>
+      </sensor>
+    </gazebo>
+  </xacro:if>
   <!-- ============================================================
        GZ SIM PLUGIN: DIFFERENTIAL DRIVE
@@ -243,5 +329,9 @@
       <left_joint>left_wheel_joint</left_joint>
       <right_joint>right_wheel_joint</right_joint>
-      <!-- Must match RDF yaml values -->
+      <!-- Odometry MUST use the same values as the physical joint positions
+           in this URDF, not the RDF's real-hardware values.  The sim model
+           has its own fixed geometry (0.287 m separation, 0.033 m radius)
+           and the diff-drive plugin's odometry must be self-consistent
+           with that geometry — otherwise SLAM/Nav2 break. -->
       <wheel_separation>${wheel_separation}</wheel_separation>
       <wheel_radius>${wheel_radius}</wheel_radius>
